Commit message: Created urdf to resemble balancing bot size. Still need to fix the origins of the base, imu and encoders

File: Self-Balancing-Bot-Pid/Simulation/ros2_ws/src/subscriber_publisher/urdf/balance_bot.urdf.xacro (robot description, xacro)
@@ -1,10 +1,31 @@
 <?xml version="1.0"?>
-<robot name="balance_bot" xmlns:xacro="http://ros.org/wiki/xacro">
+<robot name="balance_bot" xmlns:xacro="http://www.ros.org/wiki/xacro">
+  <!-- Material Definitions -->
+  <material name="chassis_gray">
+    <color rgba="0.5 0.5 0.5 1.0"/>
+  </material>
+  <material name="left_wheel_black">
+    <color rgba="0.1 0.1 0.1 1.0"/>
+  </material>
+  <material name="right_wheel_black">
+    <color rgba="0.1 0.1 0.1 1.0"/>
+  </material>
+  <material name="imu_blue">
+    <color rgba="0.0 0.0 1.0 1.0"/>
+  </material>
+  <material name="left_encoder_red">
+    <color rgba="1.0 0.0 0.0 1.0"/>
+  </material>
+  <material name="right_encoder_green">
+    <color rgba="0.0 1.0 0.0 1.0"/>
+  </material>
   <!-- Parameters -->
-  <xacro:property name="wheel_radius" value="0.05"/>
-  <xacro:property name="wheel_width" value="0.02"/>
-  <xacro:property name="chassis_height" value="0.2"/>
-  <xacro:property name="chassis_width" value="0.1"/>
-  <xacro:property name="chassis_depth" value="0.05"/>
+  <xacro:property name="wheel_radius" value="0.15"/> <!-- 3x bigger -->
+  <xacro:property name="wheel_width" value="0.06"/> <!-- 3x bigger -->
+  <xacro:property name="chassis_height" value="0.6"/> <!-- 3x bigger -->
+  <xacro:property name="chassis_width" value="0.3"/> <!-- 3x bigger -->
+  <xacro:property name="chassis_depth" value="0.15"/> <!-- 3x bigger -->
+  <xacro:property name="encoder_width" value="0.15"/> <!-- 3x bigger -->
+  <!-- <xacro:property name="encoder_radius" value="0.05"/> -->
   <!-- Chassis -->
   <link name="base_link">
@@ -13,8 +34,6 @@
         <box size="${chassis_width} ${chassis_depth} ${chassis_height}"/>
       </geometry>
-      <origin xyz="0 0 ${chassis_height/2}" rpy="0 0 0"/>
-      <material name="gray">
-        <color rgba="0.5 0.5 0.5 1.0"/>
-      </material>
+      <origin xyz="${chassis_width/2} ${chassis_depth/2} ${chassis_height/2}" rpy="0 0 1.5708"/> <!-- Position chassis at wheel height -->
+      <material name="chassis_gray"/>
     </visual>
     <collision>
@@ -22,5 +41,5 @@
         <box size="${chassis_width} ${chassis_depth} ${chassis_height}"/>
       </geometry>
-      <origin xyz="0 0 ${chassis_height/2}" rpy="0 0 0"/>
+      <origin xyz="${chassis_width/2} ${chassis_depth/2} ${chassis_height/2}" rpy="0 0 1.5708"/> <!-- Position chassis at wheel height -->
     </collision>
     <inertial>
@@ -29,8 +48,8 @@
                iyy="0.01" iyz="0.0"
                izz="0.01"/>
-      <origin xyz="0 0 ${chassis_height/2}" rpy="0 0 0"/>
+      <origin xyz="${chassis_width/2} ${chassis_depth/2} ${chassis_height/2}" rpy="0 0 1.5708"/> <!-- Position chassis at wheel height -->
     </inertial>
   </link>
-  <!-- Left wheel -->
+  <!-- Left Wheel -->
   <link name="left_wheel">
     <visual>
@@ -38,8 +57,6 @@
         <cylinder radius="${wheel_radius}" length="${wheel_width}"/>
       </geometry>
-      <origin xyz="0 ${chassis_width/2 + wheel_width/2} 0" rpy="0 1.5708 0"/>
-      <material name="black">
-        <color rgba="0 0 0 1.0"/>
-      </material>
+      <origin xyz="0 0 ${wheel_width/2}" rpy="1.5708 0 0"/>
+      <material name="left_wheel_black"/>
     </visual>
     <collision>
@@ -47,5 +64,5 @@
         <cylinder radius="${wheel_radius}" length="${wheel_width}"/>
       </geometry>
-      <origin xyz="0 ${chassis_width/2 + wheel_width/2} 0" rpy="0 1.5708 0"/>
+      <origin xyz="0 0 ${wheel_width/2}" rpy="1.5708 0 0"/>
     </collision>
     <inertial>
@@ -56,5 +73,5 @@
     </inertial>
   </link>
-  <!-- Right wheel -->
+  <!-- Right Wheel -->
   <link name="right_wheel">
     <visual>
@@ -62,6 +79,6 @@
         <cylinder radius="${wheel_radius}" length="${wheel_width}"/>
       </geometry>
-      <origin xyz="0 -${chassis_width/2 + wheel_width/2} 0" rpy="0 1.5708 0"/>
-      <material name="black"/>
+      <origin xyz="0 0 ${wheel_width/2}" rpy="1.5708 0 0"/>
+      <material name="right_wheel_black"/>
     </visual>
     <collision>
@@ -69,5 +86,5 @@
         <cylinder radius="${wheel_radius}" length="${wheel_width}"/>
       </geometry>
-      <origin xyz="0 -${chassis_width/2 + wheel_width/2} 0" rpy="0 1.5708 0"/>
+      <origin xyz="0 0 ${wheel_width/2}" rpy="1.5708 0 0"/>
     </collision>
     <inertial>
@@ -78,27 +95,25 @@
     </inertial>
   </link>
-  <!-- Wheel joints -->
+  <!-- Wheel Joints -->
   <joint name="left_wheel_joint" type="continuous">
-    <parent link="base_link"/>
-    <child link="left_wheel"/>
-    <origin xyz="0 ${chassis_width/2 + wheel_width/2} 0" rpy="0 0 0"/>
-    <axis xyz="0 1 0"/>
-  </joint>
-  <joint name="right_wheel_joint" type="continuous">
-    <parent link="base_link"/>
-    <child link="right_wheel"/>
-    <origin xyz="0 -${chassis_width/2 + wheel_width/2} 0" rpy="0 0 0"/>
-    <axis xyz="0 1 0"/>
-  </joint>
+  <parent link="base_link"/>
+  <child link="left_wheel"/>
+  <origin xyz="0 0 ${wheel_radius}" rpy="0 0 0"/> <!-- Attach wheel to side of chassis -->
+  <axis xyz="0 1 0"/>
+</joint>
+<joint name="right_wheel_joint" type="continuous">
+  <parent link="base_link"/>
+  <child link="right_wheel"/>
+  <origin xyz="0 0 ${wheel_radius}" rpy="0 0 0"/> <!-- Attach wheel to side of chassis -->
+  <axis xyz="0 1 0"/>
+</joint>
   <!-- IMU -->
   <link name="imu_link">
     <visual>
       <geometry>
-        <box size="0.02 0.02 0.02"/>
+        <box size="0.05 0.05 0.05"/>
       </geometry>
-      <origin xyz="0 0 ${chassis_height}" rpy="0 0 0"/>
-      <material name="blue">
-        <color rgba="0 0 1.0 1.0"/>
-      </material>
+      <origin xyz="0 0 0" rpy="0 0 0"/>
+      <material name="imu_blue"/>
     </visual>
   </link>
@@ -106,18 +121,34 @@
     <parent link="base_link"/>
     <child link="imu_link"/>
-    <origin xyz="0 0 ${chassis_height}" rpy="0 0 0"/>
+    <origin xyz="0 0 0.15" rpy="0 0 0"/>
   </joint>
-  <!-- Encoders on motors (fixed joints) -->
-  <link name="left_encoder"/>
-  <joint name="left_encoder_joint" type="fixed">
-    <parent link="left_wheel"/>
-    <child link="left_encoder"/>
-    <origin xyz="0 0 0" rpy="0 0 0"/>
-  </joint>
-  <link name="right_encoder"/>
-  <joint name="right_encoder_joint" type="fixed">
-    <parent link="right_wheel"/>
-    <child link="right_encoder"/>
-    <origin xyz="0 0 0" rpy="0 0 0"/>
-  </joint>
+  <!-- Encoders -->
+  <link name="left_encoder">
+  <visual>
+    <geometry>
+      <cylinder radius="0.07" length="0.03"/>
+    </geometry> <!--chassis_height chassis_width chassis_depth-->
+    <origin xyz="0 ${chassis_width/4} ${wheel_radius/2}" rpy="1.5708 0 0"/> <!-- Just behind the left wheel, sharing the same axis -->
+    <material name="left_encoder_red"/>
+  </visual>
+</link>
+<joint name="left_encoder_to_chassis_joint" type="fixed">
+  <parent link="base_link"/> <!-- Attach to the chassis -->
+  <child link="left_encoder"/> <!-- Connect to the left encoder -->
+  <origin xyz="0 ${chassis_width/4} ${wheel_radius/2}" rpy="0 0 0"/> <!-- No offset or rotation -->
+</joint>
+  <link name="right_encoder">
+    <visual>
+      <geometry>
+        <cylinder radius="0.07" length="0.03"/>
+      </geometry>
+      <origin xyz="0 ${-chassis_width/4} ${wheel_radius/2}" rpy="1.5708 0 0"/> <!-- Align with wheel -->
+      <material name="right_encoder_green"/>
+    </visual>
+  </link>
+<joint name="right_encoder_to_chassis_joint" type="fixed">
+  <parent link="base_link"/> <!-- Attach to the chassis -->
+  <child link="right_encoder"/> <!-- Connect to the right encoder -->
+  <origin xyz="0 ${-chassis_width/4} ${wheel_radius/2}" rpy="0 0 0"/> <!-- No offset or rotation -->
+</joint>
 </robot>

Commit message: Completed full URDF with correct transforms

File: Self-Balancing-Bot-Pid/Simulation/ros2_ws/src/subscriber_publisher/urdf/balance_bot.urdf.xacro (robot description, xacro)
@@ -34,12 +34,12 @@
         <box size="${chassis_width} ${chassis_depth} ${chassis_height}"/>
       </geometry>
-      <origin xyz="${chassis_width/2} ${chassis_depth/2} ${chassis_height/2}" rpy="0 0 1.5708"/> <!-- Position chassis at wheel height -->
+      <origin xyz="0 0 0" rpy="0 0 1.5708"/> <!-- Position chassis at wheel height -->
       <material name="chassis_gray"/>
     </visual>
     <collision>
       <geometry>
-        <box size="${chassis_width} ${chassis_depth} ${chassis_height}"/>
+        <box size="0 0 0"/>
       </geometry>
-      <origin xyz="${chassis_width/2} ${chassis_depth/2} ${chassis_height/2}" rpy="0 0 1.5708"/> <!-- Position chassis at wheel height -->
+      <origin xyz="0 0 0" rpy="0 0 1.5708"/> <!-- Position chassis at wheel height -->
     </collision>
     <inertial>
@@ -48,5 +48,5 @@
                iyy="0.01" iyz="0.0"
                izz="0.01"/>
-      <origin xyz="${chassis_width/2} ${chassis_depth/2} ${chassis_height/2}" rpy="0 0 1.5708"/> <!-- Position chassis at wheel height -->
+      <origin xyz="0 0 0" rpy="0 0 0"/> <!-- Position chassis at wheel height -->
     </inertial>
   </link>
@@ -57,5 +57,5 @@
         <cylinder radius="${wheel_radius}" length="${wheel_width}"/>
       </geometry>
-      <origin xyz="0 0 ${wheel_width/2}" rpy="1.5708 0 0"/>
+      <origin xyz="0 0 0" rpy="1.5708 0 0"/>
       <material name="left_wheel_black"/>
     </visual>
@@ -64,5 +64,5 @@
         <cylinder radius="${wheel_radius}" length="${wheel_width}"/>
       </geometry>
-      <origin xyz="0 0 ${wheel_width/2}" rpy="1.5708 0 0"/>
+      <origin xyz="0 0 0" rpy="1.5708 0 0"/>
     </collision>
     <inertial>
@@ -79,5 +79,5 @@
         <cylinder radius="${wheel_radius}" length="${wheel_width}"/>
       </geometry>
-      <origin xyz="0 0 ${wheel_width/2}" rpy="1.5708 0 0"/>
+      <origin xyz="0 0 0" rpy="1.5708 0 0"/>
       <material name="right_wheel_black"/>
     </visual>
@@ -86,5 +86,5 @@
         <cylinder radius="${wheel_radius}" length="${wheel_width}"/>
       </geometry>
-      <origin xyz="0 0 ${wheel_width/2}" rpy="1.5708 0 0"/>
+      <origin xyz="0 0 0" rpy="1.5708 0 0"/>
     </collision>
     <inertial>
@@ -99,5 +99,5 @@
   <parent link="base_link"/>
   <child link="left_wheel"/>
-  <origin xyz="0 0 ${wheel_radius}" rpy="0 0 0"/> <!-- Attach wheel to side of chassis -->
+  <origin xyz="0 ${chassis_width/2 + wheel_width/2 + encoder_width/2} -${chassis_height/2}" rpy="0 0 0"/> <!-- Align wheel center with bottom of chassis -->
   <axis xyz="0 1 0"/>
 </joint>
@@ -105,5 +105,5 @@
   <parent link="base_link"/>
   <child link="right_wheel"/>
-  <origin xyz="0 0 ${wheel_radius}" rpy="0 0 0"/> <!-- Attach wheel to side of chassis -->
+  <origin xyz="0 -${chassis_width/2 + wheel_width/2 + encoder_width/2} -${chassis_height/2}" rpy="0 0 0"/> <!-- Align wheel center with bottom of chassis -->
   <axis xyz="0 1 0"/>
 </joint>
@@ -129,5 +129,5 @@
       <cylinder radius="0.07" length="0.03"/>
     </geometry> <!--chassis_height chassis_width chassis_depth-->
-    <origin xyz="0 ${chassis_width/4} ${wheel_radius/2}" rpy="1.5708 0 0"/> <!-- Just behind the left wheel, sharing the same axis -->
+    <origin xyz="0 0 0" rpy="1.5708 0 0"/> <!-- Just behind the left wheel, sharing the same axis -->
     <material name="left_encoder_red"/>
   </visual>
@@ -136,5 +136,5 @@
   <parent link="base_link"/> <!-- Attach to the chassis -->
   <child link="left_encoder"/> <!-- Connect to the left encoder -->
-  <origin xyz="0 ${chassis_width/4} ${wheel_radius/2}" rpy="0 0 0"/> <!-- No offset or rotation -->
+  <origin xyz="0 ${chassis_width/2 + wheel_width/2} -${chassis_height/2}" rpy="0 0 0"/> <!-- No offset or rotation -->
 </joint>
   <link name="right_encoder">
@@ -143,5 +143,5 @@
         <cylinder radius="0.07" length="0.03"/>
       </geometry>
-      <origin xyz="0 ${-chassis_width/4} ${wheel_radius/2}" rpy="1.5708 0 0"/> <!-- Align with wheel -->
+      <origin xyz="0 0 0" rpy="1.5708 0 0"/> <!-- Align with wheel -->
       <material name="right_encoder_green"/>
     </visual>
@@ -150,5 +150,5 @@
   <parent link="base_link"/> <!-- Attach to the chassis -->
   <child link="right_encoder"/> <!-- Connect to the right encoder -->
-  <origin xyz="0 ${-chassis_width/4} ${wheel_radius/2}" rpy="0 0 0"/> <!-- No offset or rotation -->
+  <origin xyz="0 -${chassis_width/2 + wheel_width/2} -${chassis_height/2}" rpy="0 0 0"/> <!-- No offset or rotation -->
 </joint>
 </robot>

Commit message: realigned IMU

File: Self-Balancing-Bot-Pid/Simulation/ros2_ws/src/subscriber_publisher/urdf/balance_bot.urdf.xacro (robot description, xacro)
@@ -121,5 +121,5 @@
     <parent link="base_link"/>
     <child link="imu_link"/>
-    <origin xyz="0 0 0.15" rpy="0 0 0"/>
+    <origin xyz="0 0 -${chassis_height/2}" rpy="0 0 0"/>
   </joint>
   <!-- Encoders -->

Commit message: My model loads in Gazebo! I also defined the mock hardware interface for the encoders and IMU.

File: Self-Balancing-Bot-Pid/Simulation/ros2_ws/src/subscriber_publisher/urdf/balance_bot.urdf.xacro (robot description, xacro)
@@ -39,5 +39,5 @@
     <collision>
       <geometry>
-        <box size="0 0 0"/>
+        <box size="${chassis_width} ${chassis_depth} ${chassis_height}"/>
       </geometry>
       <origin xyz="0 0 0" rpy="0 0 1.5708"/> <!-- Position chassis at wheel height -->
@@ -152,3 +152,65 @@
   <origin xyz="0 -${chassis_width/2 + wheel_width/2} -${chassis_height/2}" rpy="0 0 0"/> <!-- No offset or rotation -->
 </joint>
+<!-- Gazebo Plugins -->
+  <gazebo>
+    <plugin name="imu_plugin" filename="libgazebo_ros_imu.so">
+      <ros>
+        <namespace>/imu</namespace>
+        <remapping>imu/data:=/imu/data</remapping>
+      </ros>
+      <update_rate>50</update_rate>
+      <body_name>imu_link</body_name>
+    </plugin>
+  </gazebo>
+  <gazebo>
+    <plugin name="gazebo_ros2_control" filename="libgazebo_ros2_control.so"/>
+    <robotParam>robot_description</robotParam>
+  </gazebo>
+  <!-- Transmissions -->
+  <transmission name="left_wheel_transmission">
+    <type>transmission_interface/SimpleTransmission</type>
+    <joint name="left_wheel_joint">
+      <hardwareInterface>EffortJointInterface</hardwareInterface>
+    </joint>
+    <actuator name="left_wheel_motor">
+      <mechanicalReduction>1</mechanicalReduction>
+    </actuator>
+  </transmission>
+  <transmission name="right_wheel_transmission">
+    <type>transmission_interface/SimpleTransmission</type>
+    <joint name="right_wheel_joint">
+      <hardwareInterface>EffortJointInterface</hardwareInterface>
+    </joint>
+    <actuator name="right_wheel_motor">
+      <mechanicalReduction>1</mechanicalReduction>
+    </actuator>
+  </transmission>
+  <!-- ros2_control Configuration -->
+  <ros2_control name="BalanceBotHardware" type="system">
+    <hardware>
+      <plugin>gazebo_ros2_control/GazeboSystem</plugin>
+    </hardware>
+    <joint name="left_wheel_joint">
+      <command_interface name="effort"/>
+      <state_interface name="position"/>
+      <state_interface name="velocity"/>
+    </joint>
+    <joint name="right_wheel_joint">
+      <command_interface name="effort"/>
+      <state_interface name="position"/>
+      <state_interface name="velocity"/>
+    </joint>
+    <sensor name="imu_sensor">
+      <state_interface name="orientation.x"/>
+      <state_interface name="orientation.y"/>
+      <state_interface name="orientation.z"/>
+      <state_interface name="orientation.w"/>
+      <state_interface name="angular_velocity.x"/>
+      <state_interface name="angular_velocity.y"/>
+      <state_interface name="angular_velocity.z"/>
+      <state_interface name="linear_acceleration.x"/>
+      <state_interface name="linear_acceleration.y"/>
+      <state_interface name="linear_acceleration.z"/>
+    </sensor>
+  </ros2_control>
 </robot>

Commit message: Slowing correcting the left and right wheel controllers. Focusing on the last couple dependency issues

File: Self-Balancing-Bot-Pid/Simulation/ros2_ws/src/subscriber_publisher/urdf/balance_bot.urdf.xacro (robot description, xacro)
@@ -1,4 +1,6 @@
 <?xml version="1.0"?>
 <robot name="balance_bot" xmlns:xacro="http://www.ros.org/wiki/xacro">
+  <!-- Declare the config_file parameter -->
+  <xacro:arg name="config_file" default="" />
   <!-- Material Definitions -->
   <material name="chassis_gray">
@@ -117,4 +119,14 @@
       <material name="imu_blue"/>
     </visual>
+    <!-- Add collision and inertial properties -->
+    <collision>
+      <geometry>
+        <box size="0.05 0.05 0.05"/>
+      </geometry>
+    </collision>
+    <inertial>
+      <mass value="0.01"/>
+      <inertia ixx="0.0001" ixy="0.0" ixz="0.0" iyy="0.0001" iyz="0.0" izz="0.0001"/>
+    </inertial>
   </link>
   <joint name="imu_joint" type="fixed">
@@ -164,7 +176,10 @@
   </gazebo>
   <gazebo>
-    <plugin name="gazebo_ros2_control" filename="libgazebo_ros2_control.so"/>
-    <robotParam>robot_description</robotParam>
-  </gazebo>
+  <plugin name="gazebo_ros2_control" filename="libgazebo_ros2_control.so">
+    <robot_param>robot_description</robot_param>
+    <robot_param_node>robot_state_publisher</robot_param_node>
+    <parameters>$(arg config_file)</parameters>
+  </plugin>
+</gazebo>
   <!-- Transmissions -->
   <transmission name="left_wheel_transmission">
