Commit message: Split all simulation components into different files. Figuring out if the Urdf or control laws are not correct

File: Self-Balancing-Bot-Pid/PyBullet-SImulation/balance_bot.urdf (robot description, URDF)
Before this commit: robot balance_bot, 4 links, 3 joints
Links:
- link base_link: mass 1.0 -> 0.8
- link left_wheel: mass 0.2 -> 0.1
- link right_wheel: mass 0.2 -> 0.1
Joints:
- joint left_wheel_joint: limit (none) -> lower=0.0 upper=0.548 effort=1000.0 velocity=0.0
- joint right_wheel_joint: limit (none) -> lower=0.0 upper=0.548 effort=1000.0 velocity=0.0

Commit message: Tuned the PID controller! Now I must thoroughly document all simulation code.

File: Self-Balancing-Bot-Pid/PyBullet-SImulation/balance_bot.urdf (robot description, URDF)
Before this commit: robot balance_bot, 4 links, 3 joints
Links:
- link base_link: mass 0.8 -> 0.514; geometry collision box size=0.1 0.037 0.171; visual box size=0.1 0.037 0.171
- link imu_link: geometry collision box size=0.05 0.05 0.05; visual box size=0.03 0.03 0.03
- link left_wheel: mass 0.1 -> 0.032; geometry collision cylinder length=0.026 radius=0.034; visual cylinder length=0.026 radius=0.034
- link right_wheel: mass 0.1 -> 0.032; geometry collision cylinder length=0.026 radius=0.034; visual cylinder length=0.026 radius=0.034
Joints:
- joint imu_joint: origin xyz=0 0 -0.3 rpy=0 0 0 -> xyz=0 0 0.034 rpy=0 0 0
- joint left_wheel_joint: axis 0 1 0 -> -1 0 0; limit lower=0.0 upper=0.548 effort=1000.0 velocity=0.0 -> lower=0.0 upper=0.548 effort=5.0 velocity=0.0; origin xyz=0 0.225 -0.3 rpy=0 0 0 -> xyz=-0.074 0.0 0.034 rpy=0 0 0
- joint right_wheel_joint: axis 0 1 0 -> 1 0 0; limit lower=0.0 upper=0.548 effort=1000.0 velocity=0.0 -> lower=0.0 upper=0.548 effort=5.0 velocity=0.0; origin xyz=0 -0.225 -0.3 rpy=0 0 0 -> xyz=0.074 0.0 0.034 rpy=0 0 0
