Commit message: Removed uneeded starter files. Stabilized urdf model. Fixed issue with gazebo_ros2_control not being initialized properly.

File: Self-Balancing-Bot-Pid/ROS_Simulation/ros2_ws/src/balance_bot/urdf/balance_bot.urdf.xacro (robot description, xacro)
@@ -1,34 +1,10 @@
-<?xml version="1.0"?>
 <robot name="balance_bot" xmlns:xacro="http://www.ros.org/wiki/xacro">
-  <!-- Declare the config_file parameter -->
   <xacro:arg name="config_file" default="" />
-  <!-- Material Definitions -->
-  <material name="chassis_gray">
-    <color rgba="0.5 0.5 0.5 1.0"/>
-  </material>
-  <material name="left_wheel_black">
-    <color rgba="0.1 0.1 0.1 1.0"/>
-  </material>
-  <material name="right_wheel_black">
-    <color rgba="0.1 0.1 0.1 1.0"/>
-  </material>
-  <material name="imu_blue">
-    <color rgba="0.0 0.0 1.0 1.0"/>
-  </material>
-  <material name="left_encoder_red">
-    <color rgba="1.0 0.0 0.0 1.0"/>
-  </material>
-  <material name="right_encoder_green">
-    <color rgba="0.0 1.0 0.0 1.0"/>
-  </material>
-  <!-- Parameters -->
-  <xacro:property name="wheel_radius" value="0.15"/> <!-- 3x bigger -->
-  <xacro:property name="wheel_width" value="0.06"/> <!-- 3x bigger -->
-  <xacro:property name="chassis_height" value="0.6"/> <!-- 3x bigger -->
-  <xacro:property name="chassis_width" value="0.3"/> <!-- 3x bigger -->
-  <xacro:property name="chassis_depth" value="0.15"/> <!-- 3x bigger -->
-  <xacro:property name="encoder_width" value="0.15"/> <!-- 3x bigger -->
-  <!-- <xacro:property name="encoder_radius" value="0.05"/> -->
-  <!-- Chassis -->
+  <xacro:property name="wheel_radius"   value="0.15"/>
+  <xacro:property name="wheel_width"    value="0.06"/>
+  <xacro:property name="chassis_height" value="0.6"/>
+  <xacro:property name="chassis_width"  value="0.3"/>
+  <xacro:property name="chassis_depth"  value="0.15"/>
+  <!-- ── Chassis ──────────────────────────────────────────────────────── -->
   <link name="base_link">
     <visual>
@@ -36,6 +12,5 @@
         <box size="${chassis_width} ${chassis_depth} ${chassis_height}"/>
       </geometry>
-      <origin xyz="0 0 0" rpy="0 0 1.5708"/> <!-- Position chassis at wheel height -->
-      <material name="chassis_gray"/>
+      <origin xyz="0 0 0" rpy="0 0 1.5708"/>
     </visual>
     <collision>
@@ -43,15 +18,15 @@
         <box size="${chassis_width} ${chassis_depth} ${chassis_height}"/>
       </geometry>
-      <origin xyz="0 0 0" rpy="0 0 1.5708"/> <!-- Position chassis at wheel height -->
+      <origin xyz="0 0 0" rpy="0 0 1.5708"/>
     </collision>
     <inertial>
       <mass value="1.0"/>
-      <inertia ixx="0.01" ixy="0.0" ixz="0.0"
-               iyy="0.01" iyz="0.0"
-               izz="0.01"/>
-      <origin xyz="0 0 0" rpy="0 0 0"/> <!-- Position chassis at wheel height -->
-    </inertial>
-  </link>
-  <!-- Left Wheel -->
+      <inertia ixx="0.0319" ixy="0.0" ixz="0.0"
+               iyy="0.0375" iyz="0.0"
+               izz="0.0094"/>
+      <origin xyz="0 0 0" rpy="0 0 0"/>
+    </inertial>
+  </link>
+  <!-- ── Left Wheel ───────────────────────────────────────────────────── -->
   <link name="left_wheel">
     <visual>
@@ -60,5 +35,4 @@
       </geometry>
       <origin xyz="0 0 0" rpy="1.5708 0 0"/>
-      <material name="left_wheel_black"/>
     </visual>
     <collision>
@@ -70,47 +44,65 @@
     <inertial>
       <mass value="0.2"/>
-      <inertia ixx="0.001" ixy="0.0" ixz="0.0"
-               iyy="0.001" iyz="0.0"
-               izz="0.001"/>
-    </inertial>
-  </link>
-  <!-- Right Wheel -->
-  <link name="right_wheel">
-    <visual>
-      <geometry>
-        <cylinder radius="${wheel_radius}" length="${wheel_width}"/>
-      </geometry>
-      <origin xyz="0 0 0" rpy="1.5708 0 0"/>
-      <material name="right_wheel_black"/>
-    </visual>
-    <collision>
-      <geometry>
-        <cylinder radius="${wheel_radius}" length="${wheel_width}"/>
-      </geometry>
-      <origin xyz="0 0 0" rpy="1.5708 0 0"/>
-    </collision>
-    <inertial>
-      <mass value="0.2"/>
-      <inertia ixx="0.001" ixy="0.0" ixz="0.0"
-               iyy="0.001" iyz="0.0"
-               izz="0.001"/>
-    </inertial>
-  </link>
-  <!-- Wheel Joints -->
+      <inertia ixx="0.00119" ixy="0.0" ixz="0.0"
+               iyy="0.00119" iyz="0.0"
+               izz="0.00225"/>
+    </inertial>
+  </link>
   <joint name="left_wheel_joint" type="continuous">
     <parent link="base_link"/>
     <child link="left_wheel"/>
-    <origin xyz="0 ${chassis_width/2 + wheel_width/2 + encoder_width/2} -${chassis_height/2}" rpy="0 0 0"/> <!-- Align wheel center with bottom of chassis -->
+    <origin xyz="0 ${chassis_width/2 + wheel_width/2} -${chassis_height/2}" rpy="0 0 0"/>
     <axis xyz="0 1 0"/>
     <dynamics damping="0.1" friction="0.05"/>
+    <limit effort="10.0" velocity="100.0"/>
   </joint>
+  <!-- ── Right Wheel ──────────────────────────────────────────────────── -->
+  <link name="right_wheel">
+    <visual>
+      <geometry>
+        <cylinder radius="${wheel_radius}" length="${wheel_width}"/>
+      </geometry>
+      <origin xyz="0 0 0" rpy="1.5708 0 0"/>
+    </visual>
+    <collision>
+      <geometry>
+        <cylinder radius="${wheel_radius}" length="${wheel_width}"/>
+      </geometry>
+      <origin xyz="0 0 0" rpy="1.5708 0 0"/>
+    </collision>
+    <inertial>
+      <mass value="0.2"/>
+      <inertia ixx="0.00119" ixy="0.0" ixz="0.0"
+               iyy="0.00119" iyz="0.0"
+               izz="0.00225"/>
+    </inertial>
+  </link>
   <joint name="right_wheel_joint" type="continuous">
     <parent link="base_link"/>
     <child link="right_wheel"/>
-    <origin xyz="0 -${chassis_width/2 + wheel_width/2 + encoder_width/2} -${chassis_height/2}" rpy="0 0 0"/> <!-- Align wheel center with bottom of chassis -->
+    <origin xyz="0 -${chassis_width/2 + wheel_width/2} -${chassis_height/2}" rpy="0 0 0"/>
     <axis xyz="0 1 0"/>
     <dynamics damping="0.1" friction="0.05"/>
+    <limit effort="10.0" velocity="100.0"/>
   </joint>
-  <!-- IMU -->
+   <!-- ── Wheel surface friction (critical for ground contact) ─────────── -->
+   <!-- Without mu/mu2, wheels have no grip and torque reaction launches    -->
+   <!-- the chassis.  mu=1.0 is rubber-on-concrete; kp/kd tune contact      -->
+   <!-- stiffness so wheels don't sink or bounce on the ground plane.        -->
+   <gazebo reference="left_wheel">
+     <mu1>1.0</mu1>
+     <mu2>1.0</mu2>
+     <kp>1e6</kp>
+     <kd>10.0</kd>
+     <minDepth>0.001</minDepth>
+   </gazebo>
+   <gazebo reference="right_wheel">
+     <mu1>1.0</mu1>
+     <mu2>1.0</mu2>
+     <kp>1e6</kp>
+     <kd>10.0</kd>
+     <minDepth>0.001</minDepth>
+   </gazebo>
+  <!-- ── IMU ──────────────────────────────────────────────────────────── -->
   <link name="imu_link">
     <visual>
@@ -119,7 +111,5 @@
       </geometry>
       <origin xyz="0 0 0" rpy="0 0 0"/>
-      <material name="imu_blue"/>
-    </visual>
-    <!-- Add collision and inertial properties -->
+    </visual>
     <collision>
       <geometry>
@@ -129,7 +119,8 @@
     <inertial>
       <mass value="0.01"/>
-      <inertia ixx="0.0001" ixy="0.0" ixz="0.0" iyy="0.0001" iyz="0.0" izz="0.0001"/>
-    </inertial>
-    <!-- Gazebo plugin info -->
+      <inertia ixx="0.0001" ixy="0.0" ixz="0.0"
+               iyy="0.0001" iyz="0.0"
+               izz="0.0001"/>
+    </inertial>
   </link>
   <joint name="imu_joint" type="fixed">
@@ -138,148 +129,94 @@
     <origin xyz="0 0 -${chassis_height/2}" rpy="0 0 0"/>
   </joint>
-  <!-- Encoders -->
-  <link name="left_encoder">
-  <visual>
-    <geometry>
-      <cylinder radius="0.07" length="0.03"/>
-    </geometry> <!--chassis_height chassis_width chassis_depth-->
-    <origin xyz="0 0 0" rpy="1.5708 0 0"/> <!-- Just behind the left wheel, sharing the same axis -->
-    <material name="left_encoder_red"/>
-  </visual>
-</link>
-<joint name="left_encoder_to_chassis_joint" type="fixed">
-  <parent link="base_link"/> <!-- Attach to the chassis -->
-  <child link="left_encoder"/> <!-- Connect to the left encoder -->
-  <origin xyz="0 ${chassis_width/2 + wheel_width/2} -${chassis_height/2}" rpy="0 0 0"/> <!-- No offset or rotation -->
-</joint>
-  <link name="right_encoder">
-    <visual>
-      <geometry>
-        <cylinder radius="0.07" length="0.03"/>
-      </geometry>
-      <origin xyz="0 0 0" rpy="1.5708 0 0"/> <!-- Align with wheel -->
-      <material name="right_encoder_green"/>
-    </visual>
-  </link>
-<joint name="right_encoder_to_chassis_joint" type="fixed">
-  <parent link="base_link"/> <!-- Attach to the chassis -->
-  <child link="right_encoder"/> <!-- Connect to the right encoder -->
-  <origin xyz="0 -${chassis_width/2 + wheel_width/2} -${chassis_height/2}" rpy="0 0 0"/> <!-- No offset or rotation -->
-</joint>
-<!-- Gazebo Plugins -->
-<gazebo reference="imu_link">
-  <sensor name="imu_sensor" type="imu">
-    <always_on>true</always_on>
-    <update_rate>100</update_rate>
-    <visualize>true</visualize>
-    <pose>0 0 0 0 0 0</pose>
-    <imu>
-      <angular_velocity>
-        <x>
-          <noise type="gaussian">
-            <mean>0.0</mean>
-            <stddev>0.0002</stddev>
-          </noise>
-        </x>
-        <y>
-          <noise type="gaussian">
-            <mean>0.0</mean>
-            <stddev>0.0002</stddev>
-          </noise>
-        </y>
-        <z>
-          <noise type="gaussian">
-            <mean>0.0</mean>
-            <stddev>0.0002</stddev>
-          </noise>
-        </z>
-      </angular_velocity>
-      <linear_acceleration>
-        <x>
-          <noise type="gaussian">
-            <mean>0.0</mean>
-            <stddev>0.017</stddev>
-          </noise>
-        </x>
-        <y>
-          <noise type="gaussian">
-            <mean>0.0</mean>
-            <stddev>0.017</stddev>
-          </noise>
-        </y>
-        <z>
-          <noise type="gaussian">
-            <mean>0.0</mean>
-            <stddev>0.017</stddev>
-          </noise>
-        </z>
-      </linear_acceleration>
-    </imu>
-    <topic>__default_topic__</topic>
-    <plugin name="imu_plugin" filename="libgazebo_ros_imu_sensor.so">
-      <bodyName>imu_link</bodyName>
-      <updateRateHZ>100.0</updateRateHZ>
-      <gaussianNoise>0.001</gaussianNoise>
-      <xyzOffset>0 0 0</xyzOffset>
-      <rpyOffset>0 0 0</rpyOffset>
-      <frameName>imu_link</frameName>
-      <initialOrientationAsReference>false</initialOrientationAsReference>
+  <!-- ── Gazebo IMU plugin ─────────────────────────────────────────────── -->
+  <gazebo reference="imu_link">
+    <sensor name="imu_sensor" type="imu">
+      <always_on>true</always_on>
+      <update_rate>100</update_rate>
+      <visualize>true</visualize>
+      <pose>0 0 0 0 0 0</pose>
+      <imu>
+        <angular_velocity>
+          <x>
+            <noise type="gaussian">
+              <mean>0.0</mean>
+              <stddev>0.0002</stddev>
+            </noise>
+          </x>
+          <y>
+            <noise type="gaussian">
+              <mean>0.0</mean>
+              <stddev>0.0002</stddev>
+            </noise>
+          </y>
+          <z>
+            <noise type="gaussian">
+              <mean>0.0</mean>
+              <stddev>0.0002</stddev>
+            </noise>
+          </z>
+        </angular_velocity>
+        <linear_acceleration>
+          <x>
+            <noise type="gaussian">
+              <mean>0.0</mean>
+              <stddev>0.017</stddev>
+            </noise>
+          </x>
+          <y>
+            <noise type="gaussian">
+              <mean>0.0</mean>
+              <stddev>0.017</stddev>
+            </noise>
+          </y>
+          <z>
+            <noise type="gaussian">
+              <mean>0.0</mean>
+              <stddev>0.017</stddev>
+            </noise>
+          </z>
+        </linear_acceleration>
+      </imu>
+      <plugin name="imu_plugin" filename="libgazebo_ros_imu_sensor.so">
+        <bodyName>imu_link</bodyName>
+        <updateRateHZ>100.0</updateRateHZ>
+        <gaussianNoise>0.001</gaussianNoise>
+        <xyzOffset>0 0 0</xyzOffset>
+        <rpyOffset>0 0 0</rpyOffset>
+        <frameName>imu_link</frameName>
+        <initialOrientationAsReference>false</initialOrientationAsReference>
+        <topicName>/imu_plugin/out</topicName>
+      </plugin>
+    </sensor>
+  </gazebo>
+  <!-- ── gazebo_ros2_control plugin ───────────────────────────────────── -->
+  <gazebo>
+    <plugin name="gazebo_ros2_control" filename="libgazebo_ros2_control.so">
+      <robot_param>robot_description</robot_param>
+      <robot_param_node>robot_state_publisher</robot_param_node>
+      <parameters>$(arg config_file)</parameters>
     </plugin>
-  </sensor>
-</gazebo>
-  <gazebo>
-  <plugin name="gazebo_ros2_control" filename="libgazebo_ros2_control.so">
-    <robot_param>robot_description</robot_param>
-    <parameters>$(arg config_file)</parameters>
-    <robot_param_node>robot_state_publisher</robot_param_node>
-     <control_period>0.001</control_period>
-  </plugin>
-</gazebo>
-  <!-- Transmissions -->
-  <transmission name="left_wheel_transmission">
-    <type>transmission_interface/SimpleTransmission</type>
-    <joint name="left_wheel_joint">
-      <hardwareInterface>hardware_interface/EffortJointInterface</hardwareInterface>
-    </joint>
-    <actuator name="left_wheel_motor">
-      <mechanicalReduction>1</mechanicalReduction>
-    </actuator>
-  </transmission>
-  <transmission name="right_wheel_transmission">
-    <type>transmission_interface/SimpleTransmission</type>
-    <joint name="right_wheel_joint">
-      <hardwareInterface>hardware_interface/EffortJointInterface</hardwareInterface>
-    </joint>
-    <actuator name="right_wheel_motor">
-      <mechanicalReduction>1</mechanicalReduction>
-    </actuator>
-  </transmission>
-  <!-- ros2_control Configuration -->
+  </gazebo>
+  <!-- ── ros2_control hardware interface ──────────────────────────────── -->
   <ros2_control name="BalanceBotHardware" type="system">
-    <hardware>
-      <plugin>gazebo_ros2_control/GazeboSystem</plugin>
-    </hardware>
-    <joint name="left_wheel_joint">
-      <command_interface name="effort"/>
-      <state_interface name="position"/>
-      <state_interface name="velocity"/>
-    </joint>
-    <joint name="right_wheel_joint">
-      <command_interface name="effort"/>
-      <state_interface name="position"/>
-      <state_interface name="velocity"/>
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