Commit message: Finsihed up controller tuning, and class restructuring for c++ code. Balance bot simulation complete!

File: Self-Balancing-Bot-Pid/ROS_Simulation/ros2_ws/src/balance_bot/urdf/balance_bot.urdf.xacro (robot description, xacro)
@@ -1,50 +1,42 @@
 <robot name="balance_bot" xmlns:xacro="http://www.ros.org/wiki/xacro">
   <xacro:arg name="config_file" default="" />
-  <xacro:property name="wheel_radius"   value="0.15"/>
-  <xacro:property name="wheel_width"    value="0.06"/>
-  <xacro:property name="chassis_height" value="0.6"/>
-  <xacro:property name="chassis_width"  value="0.3"/>
-  <xacro:property name="chassis_depth"  value="0.15"/>
-  <!-- ── Chassis ──────────────────────────────────────────────────────── -->
+  <material name="body">  <color rgba="0.5 0.5 0.5 1"/> </material>
+  <material name="wheel"> <color rgba="0.2 0.2 0.2 1"/> </material>
   <link name="base_link">
     <visual>
-      <geometry>
-        <box size="${chassis_width} ${chassis_depth} ${chassis_height}"/>
-      </geometry>
-      <origin xyz="0 0 0" rpy="0 0 1.5708"/>
+      <geometry><box size="0.1 0.037 0.171"/></geometry>
+      <origin rpy="0 0 0" xyz="0 0.0 0.0995"/>
+      <material name="body"/>
     </visual>
     <collision>
-      <geometry>
-        <box size="${chassis_width} ${chassis_depth} ${chassis_height}"/>
-      </geometry>
-      <origin xyz="0 0 0" rpy="0 0 1.5708"/>
+      <geometry><box size="0.1 0.037 0.171"/></geometry>
+      <origin rpy="0 0 0" xyz="0 0.0 0.0995"/>
     </collision>
     <inertial>
-      <mass value="1.0"/>
-      <inertia ixx="0.0319" ixy="0.0" ixz="0.0"
-               iyy="0.0375" iyz="0.0"
-               izz="0.0094"/>
-      <origin xyz="0 0 0" rpy="0 0 0"/>
+      <mass value="0.514"/>
+      <!-- ixx/iyy/izz for a uniform solid box: m*(h?+d?)/12 etc.         -->
+      <inertia ixx="0.0012568" ixy="0.0" ixz="0.0"
+               iyy="0.001311"  iyz="0.0"
+               izz="0.000487"/>
+      <!-- CoM at geometric center ? matches PyBullet URDF intent          -->
+      <origin rpy="0 0 0" xyz="0 0.0 0.0995"/>
     </inertial>
   </link>
-  <!-- ── Left Wheel ───────────────────────────────────────────────────── -->
   <link name="left_wheel">
     <visual>
-      <geometry>
-        <cylinder radius="${wheel_radius}" length="${wheel_width}"/>
-      </geometry>
-      <origin xyz="0 0 0" rpy="1.5708 0 0"/>
+      <geometry><cylinder length="0.026" radius="0.034"/></geometry>
+      <origin rpy="0 1.5707963 0" xyz="0 0 0"/>
+      <material name="wheel"/>
     </visual>
     <collision>
-      <geometry>
-        <cylinder radius="${wheel_radius}" length="${wheel_width}"/>
-      </geometry>
-      <origin xyz="0 0 0" rpy="1.5708 0 0"/>
+      <geometry><cylinder length="0.026" radius="0.034"/></geometry>
+      <origin rpy="0 1.5707963 0" xyz="0 0 0"/>
     </collision>
     <inertial>
-      <mass value="0.2"/>
-      <inertia ixx="0.00119" ixy="0.0" ixz="0.0"
-               iyy="0.00119" iyz="0.0"
-               izz="0.00225"/>
+      <mass value="0.032"/>
+      <inertia ixx="1.3E-05" ixy="0.0" ixz="0.0"
+               iyy="1.3E-05" iyz="0.0"
+               izz="2.3E-05"/>
+      <origin rpy="0 0 0" xyz="0 0 0"/>
     </inertial>
   </link>
@@ -52,28 +44,26 @@
     <parent link="base_link"/>
     <child link="left_wheel"/>
-    <origin xyz="0 ${chassis_width/2 + wheel_width/2} -${chassis_height/2}" rpy="0 0 0"/>
-    <axis xyz="0 1 0"/>
-    <dynamics damping="0.1" friction="0.05"/>
-    <limit effort="10.0" velocity="100.0"/>
+    <axis xyz="-1 0 0"/>
+    <!-- velocity=100 rad/s is a generous hardware ceiling (not a control  -->
+    <!-- limit); MAX_VEL=50 in the controller is the effective cap.         -->
+    <limit effort="25.0" velocity="100.0"/>
+    <origin rpy="0 0 0" xyz="-0.074 0.0 0.034"/>
   </joint>
-  <!-- ── Right Wheel ──────────────────────────────────────────────────── -->
   <link name="right_wheel">
     <visual>
-      <geometry>
-        <cylinder radius="${wheel_radius}" length="${wheel_width}"/>
-      </geometry>
-      <origin xyz="0 0 0" rpy="1.5708 0 0"/>
+      <geometry><cylinder length="0.026" radius="0.034"/></geometry>
+      <origin rpy="0 1.5707963 0" xyz="0 0 0"/>
+      <material name="wheel"/>
     </visual>
     <collision>
-      <geometry>
-        <cylinder radius="${wheel_radius}" length="${wheel_width}"/>
-      </geometry>
-      <origin xyz="0 0 0" rpy="1.5708 0 0"/>
+      <geometry><cylinder length="0.026" radius="0.034"/></geometry>
+      <origin rpy="0 1.5707963 0" xyz="0 0 0"/>
     </collision>
     <inertial>
-      <mass value="0.2"/>
-      <inertia ixx="0.00119" ixy="0.0" ixz="0.0"
-               iyy="0.00119" iyz="0.0"
-               izz="0.00225"/>
+      <mass value="0.032"/>
+      <inertia ixx="1.3E-05" ixy="0.0" ixz="0.0"
+               iyy="1.3E-05" iyz="0.0"
+               izz="2.3E-05"/>
+      <origin rpy="0 0 0" xyz="0 0 0"/>
     </inertial>
   </link>
@@ -81,45 +71,36 @@
     <parent link="base_link"/>
     <child link="right_wheel"/>
-    <origin xyz="0 -${chassis_width/2 + wheel_width/2} -${chassis_height/2}" rpy="0 0 0"/>
-    <axis xyz="0 1 0"/>
-    <dynamics damping="0.1" friction="0.05"/>
-    <limit effort="10.0" velocity="100.0"/>
+    <axis xyz="1 0 0"/>
+    <limit effort="25.0" velocity="100.0"/>
+    <origin rpy="0 0 0" xyz="0.074 0.0 0.034"/>
   </joint>
-   <!-- ── Wheel surface friction (critical for ground contact) ─────────── -->
-   <!-- Without mu/mu2, wheels have no grip and torque reaction launches    -->
-   <!-- the chassis.  mu=1.0 is rubber-on-concrete; kp/kd tune contact      -->
-   <!-- stiffness so wheels don't sink or bounce on the ground plane.        -->
-   <gazebo reference="left_wheel">
-     <mu1>1.0</mu1>
-     <mu2>1.0</mu2>
-     <kp>1e6</kp>
-     <kd>10.0</kd>
-     <minDepth>0.001</minDepth>
-   </gazebo>
-   <gazebo reference="right_wheel">
-     <mu1>1.0</mu1>
-     <mu2>1.0</mu2>
-     <kp>1e6</kp>
-     <kd>10.0</kd>
-     <minDepth>0.001</minDepth>
-   </gazebo>
-  <!-- ── IMU ──────────────────────────────────────────────────────────── -->
+  <gazebo reference="left_wheel">
+    <mu1>5.0</mu1>
+    <mu2>5.0</mu2>
+    <kp>1e6</kp>
+    <kd>10.0</kd>
+    <minDepth>0.001</minDepth>
+  </gazebo>
+  <gazebo reference="right_wheel">
+    <mu1>5.0</mu1>
+    <mu2>5.0</mu2>
+    <kp>1e6</kp>
+    <kd>10.0</kd>
+    <minDepth>0.001</minDepth>
+  </gazebo>
   <link name="imu_link">
     <visual>
-      <geometry>
-        <box size="0.05 0.05 0.05"/>
-      </geometry>
+      <geometry><box size="0.03 0.03 0.03"/></geometry>
       <origin xyz="0 0 0" rpy="0 0 0"/>
     </visual>
     <collision>
-      <geometry>
-        <box size="0.05 0.05 0.05"/>
-      </geometry>
+      <geometry><box size="0.05 0.05 0.05"/></geometry>
+      <origin xyz="0 0 0" rpy="0 0 0"/>
     </collision>
     <inertial>
       <mass value="0.01"/>
-      <inertia ixx="0.0001" ixy="0.0" ixz="0.0"
-               iyy="0.0001" iyz="0.0"
-               izz="0.0001"/>
+      <origin xyz="0 0 0" rpy="0 0 0"/>
+      <inertia ixx="0.0001" iyy="0.0001" izz="0.0001"
+               ixy="0.0"   ixz="0.0"   iyz="0.0"/>
     </inertial>
   </link>
@@ -127,58 +108,27 @@
     <parent link="base_link"/>
     <child link="imu_link"/>
-    <origin xyz="0 0 -${chassis_height/2}" rpy="0 0 0"/>
+    <origin xyz="0 0 0.034" rpy="0 0 0"/>
   </joint>
-  <!-- ── Gazebo IMU plugin ─────────────────────────────────────────────── -->
   <gazebo reference="imu_link">
     <sensor name="imu_sensor" type="imu">
       <always_on>true</always_on>
-      <update_rate>100</update_rate>
+      <update_rate>200</update_rate>  <!-- raised from 100 -->
       <visualize>true</visualize>
       <pose>0 0 0 0 0 0</pose>
       <imu>
         <angular_velocity>
-          <x>
-            <noise type="gaussian">
-              <mean>0.0</mean>
-              <stddev>0.0002</stddev>
-            </noise>
-          </x>
-          <y>
-            <noise type="gaussian">
-              <mean>0.0</mean>
-              <stddev>0.0002</stddev>
-            </noise>
-          </y>
-          <z>
-            <noise type="gaussian">
-              <mean>0.0</mean>
-              <stddev>0.0002</stddev>
-            </noise>
-          </z>
+          <x><noise type="gaussian"><mean>0.0</mean><stddev>0.0002</stddev></noise></x>
+          <y><noise type="gaussian"><mean>0.0</mean><stddev>0.0002</stddev></noise></y>
+          <z><noise type="gaussian"><mean>0.0</mean><stddev>0.0002</stddev></noise></z>
         </angular_velocity>
         <linear_acceleration>
-          <x>
-            <noise type="gaussian">
-              <mean>0.0</mean>
-              <stddev>0.017</stddev>
-            </noise>
-          </x>
-          <y>
-            <noise type="gaussian">
-              <mean>0.0</mean>
-              <stddev>0.017</stddev>
-            </noise>
-          </y>
-          <z>
-            <noise type="gaussian">
-              <mean>0.0</mean>
-              <stddev>0.017</stddev>
-            </noise>
-          </z>
+          <x><noise type="gaussian"><mean>0.0</mean><stddev>0.017</stddev></noise></x>
+          <y><noise type="gaussian"><mean>0.0</mean><stddev>0.017</stddev></noise></y>
+          <z><noise type="gaussian"><mean>0.0</mean><stddev>0.017</stddev></noise></z>
         </linear_acceleration>
       </imu>
       <plugin name="imu_plugin" filename="libgazebo_ros_imu_sensor.so">
         <bodyName>imu_link</bodyName>
-        <updateRateHZ>100.0</updateRateHZ>
+        <updateRateHZ>200.0</updateRateHZ>  <!-- raised from 100 -->
         <gaussianNoise>0.001</gaussianNoise>
         <xyzOffset>0 0 0</xyzOffset>
@@ -190,5 +140,4 @@
     </sensor>
   </gazebo>
-  <!-- ── gazebo_ros2_control plugin ───────────────────────────────────── -->
   <gazebo>
     <plugin name="gazebo_ros2_control" filename="libgazebo_ros2_control.so">
@@ -198,25 +147,25 @@
     </plugin>
   </gazebo>
-  <!-- ── ros2_control hardware interface ──────────────────────────────── -->
+                           -->
   <ros2_control name="BalanceBotHardware" type="system">
-      <hardware>
-        <plugin>gazebo_ros2_control/GazeboSystem</plugin>
-      </hardware>
-      <joint name="left_wheel_joint">
-        <command_interface name="effort">
-          <param name="min">-10.0</param>
-          <param name="max">10.0</param>
-        </command_interface>
-        <state_interface name="position"/>
-        <state_interface name="velocity"/>
-      </joint>
-      <joint name="right_wheel_joint">
-        <command_interface name="effort">
-          <param name="min">-10.0</param>
-          <param name="max">10.0</param>
-        </command_interface>
-        <state_interface name="position"/>
-        <state_interface name="velocity"/>
-      </joint>
-    </ros2_control>
+    <hardware>
+      <plugin>gazebo_ros2_control/GazeboSystem</plugin>
+    </hardware>
+    <joint name="left_wheel_joint">
+      <command_interface name="velocity">
+        <param name="min">-50.0</param>  <!-- rad/s; matches MAX_VEL in cpp -->
+        <param name="max"> 50.0</param>
+      </command_interface>
+      <state_interface name="position"/>
+      <state_interface name="velocity"/>
+    </joint>
+    <joint name="right_wheel_joint">
+      <command_interface name="velocity">
+        <param name="min">-50.0</param>
+        <param name="max"> 50.0</param>
+      </command_interface>
+      <state_interface name="position"/>
+      <state_interface name="velocity"/>
+    </joint>
+  </ros2_control>
 </robot>
